File: powerTimerPCB/powerTimer.kicad_sch (KiCad schematic)
At the start: 32 parts, among them J1 Conn_01x02, J2 Conn_01x06, Q1 AO3401A, Q2 S8050H, Q3 S8050H, Q4 AO3401A, Q5 AO3401A, SW1 TS-1185EC-C-D-B, U1 RV-3028-C7 32.768KHZ 1PPM TA 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

Commit message: Add JLCPCB-ready LCSC part numbers and bump silkscreen text to 0.8mm
Prepares the project for a JLCPCB populated-board order at quantity 10 by
filling in missing LCSC part numbers in the schematic and resolving the 13
text_height DRC warnings on the back silkscreen.

Schematic — 74 properties added across 21 components:

  Refs                              | Value | LCSC      | Tier
  ----------------------------------|-------|-----------|------
  C1                                | 100nF | C14663    | Basic
  C2                                | 10uF  | C19702    | Basic
  D1, D2, D3                        | LL4148| C2857181  | Ext
  Q1, Q4, Q5                        | AO3401A| C15127   | Basic
  R1, R3, R5, R6, R10, R11, R14     | 10K   | C25804    | Basic
  R2, R4, R7, R8                    | 100K  | C25803    | Basic
  R9                                | 470   | C23179    | Basic

MPN and Manufacturer fields also backfilled on every component (including
the five that already had LCSC numbers), so the schematic is now fully sourced.

PCB — proportional silkscreen bump:

13 (gr_text) entries on B.Silkscreen had (size 0.75 0.75) (thickness 0.15),
which violated the project's own silk-text-height rule of 0.8mm. They are
now (size 0.8 0.8) (thickness 0.16) — a 1.0667x proportional scale that
preserves the stroke-to-height ratio at 0.20.

DRC after the bump: 13 text_height warnings -> 0. Total DRC drops from 38 to
25 violations, with the remaining 25 all being lib_footprint_mismatch /
lib_footprint_issues — known-tolerable (custom RTCSwitchLib / HandSolder
footprint variants), no fab impact.

J1 and J2 (THT pin headers) are intentionally left without LCSC numbers;
they are hand-soldered after JLCPCB delivery since Economic Assembly is
SMD-only.

Note: powerTimer.kicad_prl change is incidental — KiCad regenerates this
per-user UI-state file on every export run. Keeping it tracked because the
repo already does so.

via [HAPI](https://hapi.run)

Co-Authored-By: HAPI <nore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
Parts:
- C1: LCSC Part (none) -> C14663; MPN (none) -> CC0603KRX7R9BB104; Manufacturer (none) -> YAGEO
- C2: LCSC Part (none) -> C19702; MPN (none) -> CL10A106KP8NNNC; Manufacturer (none) -> Samsung Electro-Mechanics
- C3: MPN (none) -> TAJA475K016RNJ; Manufacturer (none) -> AVX
- D1, D2, D3: LCSC Part (none) -> C2857181; MPN (none) -> LL4148; Manufacturer (none) -> MDD
- J1: Notes (none) -> Pin header 2.54mm 1x2 — hand-solder after JLCPCB delivery
- J2: Notes (none) -> Pin header 2.54mm 1x6 — hand-solder after JLCPCB delivery
- LED1: MPN (none) -> Green LED 0805; Manufacturer (none) -> Generic
- Q1, Q4, Q5: LCSC Part (none) -> C15127; MPN (none) -> AO3401A; Manufacturer (none) -> Alpha & Omega Semicon
- Q2, Q3: MPN (none) -> S8050H; Manufacturer (none) -> JCET
- R1, R10, R11, R14, R3, R5, R6: LCSC Part (none) -> C25804; MPN (none) -> 0603WAF1002T5E; Manufacturer (none) -> UNI-ROYAL
- R2, R4, R7, R8: LCSC Part (none) -> C25803; MPN (none) -> 0603WAF1003T5E; Manufacturer (none) -> UNI-ROYAL
- R9: LCSC Part (none) -> C23179; MPN (none) -> 0603WAF4700T5E; Manufacturer (none) -> UNI-ROYAL
- SW1: MPN (none) -> TS-1185EC-C-D-B; Manufacturer (none) -> XKB Connection
- U1: MPN (none) -> RV-3028-C7; Manufacturer (none) -> Micro Crystal
